File: LIC_rack_ZB-00.brd (EAGLE design)
At the start: 162.6 x 128.7 mm, 55 parts, among them X1 FAC32SE, X2 FAC32SE, X3 FAC32SE, X4 FAC32SE, X5 FAC32SE, X6 FAC32SE, X7 FAC32SE

Commit message: Uprava knihovny
Parts:
- moved C18 20.3 mm to (131.3, 103.8)
- moved C23 20.3 mm to (131.3, 93.6)
- moved C6 20.3 mm to (131.3, 88.5)
- moved C9 20.3 mm to (131.3, 98.7)
- moved JUM5 20.3 mm to (127.5, 35.1)
- moved JUM6 20.3 mm to (127.5, 66.9)
- moved JUM7 20.3 mm to (127.5, 92.3)
Routing:
- net MODUL_RST: track 165.0 -> 175.8 mm
- net +5V: track 295.4 -> 306.0 mm
- net SYNC01: track 164.9 -> 175.4 mm
- net -12V: track 190.6 -> 201.0 mm
- net +24V: track 191.0 -> 201.4 mm
- net SYNC15: track 164.9 -> 175.3 mm
- net SYNC11: track 164.9 -> 175.3 mm
- net SYNC09: track 164.9 -> 175.3 mm
- net SYNC07: track 164.9 -> 175.2 mm
- net SYNC05: track 164.9 -> 175.3 mm
- net EXT_RS485+: track 164.9 -> 175.3 mm
- net +12V: track 190.6 -> 201.0 mm
- net SYNC13: track 174.8 -> 185.1 mm
- net SYNC03: track 164.9 -> 175.2 mm
- net RS485+: track 165.0 -> 175.3 mm
